File: pcb/e.kicad_pcb (KiCad board)
At the start: 2 copper layers, 118 parts, among them J1 Grids and Anodes, J2 CH32V003 PROG, J3 AC 15V, J4 AC 27V, J5 AC Filament Middle, J6 Step-down IN, J7 Step-down OUT, J9 GPS Header, Q1 BC237, Q10 BC307, Q11 BC237, Q12 BC307, Q13 BC237, Q14 BC307, Q15 BC237, Q16 BC307, Q17 BC237, Q18 BC307, Q19 BC237, Q2 BC307, Q20 BC307, Q21 BC237, Q22 BC307, Q23 BC237, Q24 BC307, Q25 BC237, Q26 BC307, Q27 BC237, Q28 BC307, Q29 BC237, Q3 BC237, Q30 BC307, Q31 BC237, Q32 BC307, Q33 BC237, Q34 BC307, Q4 BC307, Q5 BC237, Q6 BC307, Q7 BC237, Q8 BC307, Q9 BC237, U1 74HC595, U2 CH32V003FxPx, U3 74HC595

Commit message: smd pcb
Parts:
- added J10: GND, Connector_PinHeader_2.54mm:PinHeader_1x01_P2.54mm_Vertical, F.Cu at (79.5, 43.5)
- added J8: DC +5V, Connector_PinHeader_2.54mm:PinHeader_1x01_P2.54mm_Vertical, F.Cu at (89.5, 43.5)
- J6: value Step-down IN -> DC +15V; footprint Connector_PinHeader_1.00mm:PinHeader_1x02_P1.00mm_Vertical -> Connector_PinHeader_2.54mm:PinHeader_1x01_P2.54mm_Vertical
- J7: value Step-down OUT -> DC 15GND; footprint Connector_PinHeader_1.00mm:PinHeader_1x02_P1.00mm_Vertical -> Connector_PinHeader_2.54mm:PinHeader_1x01_P2.54mm_Vertical
- Q1, Q11, Q13, Q15, Q17, Q19, Q21, Q23, Q25, Q27, Q29, Q3, Q31, Q33, Q5, Q7, Q9: value BC237 -> BC848; footprint Package_TO_SOT_THT:TO-92_Inline -> Package_TO_SOT_SMD:SOT-23
- Q10, Q12, Q14, Q16, Q18, Q2, Q20, Q22, Q24, Q26, Q28, Q30, Q32, Q34, Q4, Q6, Q8: value BC307 -> BC856; footprint Package_TO_SOT_THT:TO-92_Inline -> Package_TO_SOT_SMD:SOT-23
- R1, R10, R11, R12, R13, R14, R15, R16, R17, R18, R19, R2, R20, R21, R22, R23, R24, R25, R26, R27, R28, R29, R3, R30, R31, R32, R33, R34, R35, R36, R37, R38, R39, R4, R40, R41, R42, R43, R44, R45, R46, R47, R48, R49, R5, R50, R51, R52, R53, R54, R55, R56, R57, R58, R59, R6, R60, R61, R62, R63, R64, R65, R66, R67, R68, R7, R8, R9: footprint Resistor_THT:R_Axial_DIN0207_L6.3mm_D2.5mm_P10.16mm_Horizontal -> Resistor_SMD:R_0201_0603Metric
- U1, U3: value 74HC595 -> 74HC164; footprint Package_DIP:DIP-16_W7.62mm_Socket -> Package_SO:SSOP-14_5.3x6.2mm_P0.65mm
- moved R68 169.3 mm to (15.0, 60.0), turned to 180 degrees
- moved R64 159.1 mm to (15.0, 57.8), turned to 180 degrees
- moved Q34 155.1 mm to (28.6, 24.0)
- moved R67 153.0 mm to (29.6, 20.9)
- moved Q33 150.5 mm to (27.6, 29.0), turned to 90 degrees
- moved R65 150.2 mm to (27.4, 20.9)
- moved R66 149.0 mm to (28.6, 31.9)
- moved R60 148.8 mm to (15.0, 55.2), turned to 180 degrees
- moved Q32 140.1 mm to (33.6, 24.1)
- moved R56 138.6 mm to (15.0, 52.5), turned to 180 degrees
- moved R63 137.9 mm to (34.7, 20.9)
- moved Q31 135.5 mm to (32.5, 29.0), turned to 90 degrees
- moved R61 135.1 mm to (32.5, 20.9)
- moved R62 134.0 mm to (33.5, 31.9)
- moved U1 128.8 mm to (46.5, 40.1), turned to 180 degrees
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Connections:
- D1 pad 1: +3.3V -> +5V
- J6 pad 1: Net-(D2--) -> Net-(D2-+)
- J7 pad 1: Net-(D1-A) -> Net-(D2--)
- Q1 pad 1: Net-(Q1-C) -> /A_LOW
- Q1 pad 2: /A_LOW -> Net-(Q1-E)
- Q1 pad 3: Net-(Q1-E) -> Net-(Q1-C)
- Q10 pad 1: /E_HIGH -> Net-(Q10-B)
- Q10 pad 2: Net-(Q10-B) -> Net-(Q10-E)
- Q10 pad 3: Net-(Q10-E) -> /E_HIGH
- Q11 pad 1: Net-(Q11-C) -> /F_LOW
- Q11 pad 2: /F_LOW -> Net-(Q11-E)
- Q11 pad 3: Net-(Q11-E) -> Net-(Q11-C)
- Q12 pad 1: /F_HIGH -> Net-(Q11-C)
- Q12 pad 2: Net-(Q11-C) -> Net-(Q12-E)
- Q12 pad 3: Net-(Q12-E) -> /F_HIGH
- Q13 pad 1: Net-(Q13-C) -> /G_LOW
- Q13 pad 2: /G_LOW -> Net-(Q13-E)
- Q13 pad 3: Net-(Q13-E) -> Net-(Q13-C)
- Q14 pad 1: /G_HIGH -> Net-(Q13-C)
- Q14 pad 2: Net-(Q13-C) -> Net-(Q14-E)
- Q14 pad 3: Net-(Q14-E) -> /G_HIGH
- Q15 pad 1: Net-(Q15-C) -> /H_LOW
- Q15 pad 2: /H_LOW -> Net-(Q15-E)
- Q15 pad 3: Net-(Q15-E) -> Net-(Q15-C)
- Q16 pad 1: /H_HIGH -> Net-(Q15-C)
- Q16 pad 2: Net-(Q15-C) -> Net-(Q16-E)
- Q16 pad 3: Net-(Q16-E) -> /H_HIGH
- Q17 pad 1: Net-(Q17-C) -> /SEG1_LOW
- Q17 pad 2: /SEG1_LOW -> Net-(Q17-E)
- Q17 pad 3: Net-(Q17-E) -> Net-(Q17-C)
- Q18 pad 1: /SEG1_HIGH -> Net-(Q17-C)
- Q18 pad 2: Net-(Q17-C) -> Net-(Q18-E)
- Q18 pad 3: Net-(Q18-E) -> /SEG1_HIGH
- Q19 pad 1: Net-(Q19-C) -> /SEG2_LOW
- Q19 pad 2: /SEG2_LOW -> Net-(Q19-E)
- Q19 pad 3: Net-(Q19-E) -> Net-(Q19-C)
- Q2 pad 1: /A_HIGH -> Net-(Q1-C)
- Q2 pad 2: Net-(Q1-C) -> Net-(Q2-E)
- Q2 pad 3: Net-(Q2-E) -> /A_HIGH
- Q20 pad 1: /SEG1_HIGH -> Net-(Q19-C)
- Q20 pad 2: Net-(Q19-C) -> Net-(Q20-E)
- Q20 pad 3: Net-(Q20-E) -> /SEG2_HIGH
- Q21 pad 1: Net-(Q21-C) -> /SEG3_LOW
- Q21 pad 2: /SEG3_LOW -> Net-(Q21-E)
- Q21 pad 3: Net-(Q21-E) -> Net-(Q21-C)
- Q22 pad 1: /SEG3_HIGH -> Net-(Q21-C)
- Q22 pad 2: Net-(Q21-C) -> Net-(Q22-E)
- Q22 pad 3: Net-(Q22-E) -> /SEG3_HIGH
- Q23 pad 1: Net-(Q23-C) -> /SEG4_LOW
- Q23 pad 2: /SEG4_LOW -> Net-(Q23-E)
- Q23 pad 3: Net-(Q23-E) -> Net-(Q23-C)
- Q24 pad 1: /SEG4_HIGH -> Net-(Q23-C)
- Q24 pad 2: Net-(Q23-C) -> Net-(Q24-E)
- Q24 pad 3: Net-(Q24-E) -> /SEG4_HIGH
- Q25 pad 1: Net-(Q25-C) -> /SEG5_LOW
- Q25 pad 2: /SEG5_LOW -> Net-(Q25-E)
- Q25 pad 3: Net-(Q25-E) -> Net-(Q25-C)
- Q26 pad 1: /SEG5_HIGH -> Net-(Q25-C)
- Q26 pad 2: Net-(Q25-C) -> Net-(Q26-E)
- Q26 pad 3: Net-(Q26-E) -> /SEG5_HIGH
- Q27 pad 1: Net-(Q27-C) -> /SEG6_LOW
- Q27 pad 2: /SEG6_LOW -> Net-(Q27-E)
- Q27 pad 3: Net-(Q27-E) -> Net-(Q27-C)
- Q28 pad 1: /SEG6_HIGH -> Net-(Q27-C)
- Q28 pad 2: Net-(Q27-C) -> Net-(Q28-E)
- Q28 pad 3: Net-(Q28-E) -> /SEG6_HIGH
- Q29 pad 1: Net-(Q29-C) -> /SEG7_LOW
- Q29 pad 2: /SEG7_LOW -> Net-(Q29-E)
- Q29 pad 3: Net-(Q29-E) -> Net-(Q29-C)
- Q3 pad 1: Net-(Q3-C) -> /B_LOW
- Q3 pad 2: /B_LOW -> Net-(Q3-E)
- Q3 pad 3: Net-(Q3-E) -> Net-(Q3-C)
- Q30 pad 1: /SEG7_HIGH -> Net-(Q29-C)
- Q30 pad 2: Net-(Q29-C) -> Net-(Q30-E)
- Q30 pad 3: Net-(Q30-E) -> /SEG7_HIGH
- Q31 pad 1: Net-(Q31-C) -> /SEG8_LOW
- Q31 pad 2: /SEG8_LOW -> Net-(Q31-E)
- Q31 pad 3: Net-(Q31-E) -> Net-(Q31-C)
- Q32 pad 1: /SEG8_HIGH -> Net-(Q31-C)
- Q32 pad 2: Net-(Q31-C) -> Net-(Q32-E)
- Q32 pad 3: Net-(Q32-E) -> /SEG8_HIGH
- Q33 pad 1: Net-(Q33-C) -> /SEG9_LOW
- Q33 pad 2: /SEG9_LOW -> Net-(Q33-E)
- Q33 pad 3: Net-(Q33-E) -> Net-(Q33-C)
- Q34 pad 1: /SEG9_HIGH -> Net-(Q33-C)
- Q34 pad 2: Net-(Q33-C) -> Net-(Q34-E)
- Q34 pad 3: Net-(Q34-E) -> /SEG9_HIGH
- Q4 pad 1: /B_HIGH -> Net-(Q3-C)
- Q4 pad 2: Net-(Q3-C) -> Net-(Q4-E)
- Q4 pad 3: Net-(Q4-E) -> /B_HIGH
- Q5 pad 1: Net-(Q5-C) -> /C_LOW
- Q5 pad 2: /C_LOW -> Net-(Q5-E)
- Q5 pad 3: Net-(Q5-E) -> Net-(Q5-C)
- Q6 pad 1: /C_HIGH -> Net-(Q5-C)
- Q6 pad 2: Net-(Q5-C) -> Net-(Q6-E)
- Q6 pad 3: Net-(Q6-E) -> /C_HIGH
- Q7 pad 1: Net-(Q7-C) -> /D_LOW
- Q7 pad 2: /D_LOW -> Net-(Q7-E)
- Q7 pad 3: Net-(Q7-E) -> Net-(Q7-C)
- Q8 pad 1: /D_HIGH -> Net-(Q7-C)
- Q8 pad 2: Net-(Q7-C) -> Net-(Q8-E)
- Q8 pad 3: Net-(Q8-E) -> /D_HIGH
- Q9 pad 1: Net-(Q10-B) -> /E_LOW
- Q9 pad 2: /E_LOW -> Net-(Q9-E)
- Q9 pad 3: Net-(Q9-E) -> Net-(Q10-B)
- R40 pad 1: /SEG1_HIGH -> /SEG2_HIGH
- U1 pad 1: /SEG2_LOW -> /SER
- U1 pad 10: +5V -> /SEG6_LOW
- U1 pad 11: /SRCLK -> /SEG7_LOW
- U1 pad 12: /SRCLK -> /SEG8_LOW
- U1 pad 13: GND -> unconnected-(U1-Q7-Pad13)
- U1 pad 14: /SER -> +5V
- U1 pad 2: /SEG3_LOW -> +5V
- U1 pad 3: /SEG4_LOW -> /SEG2_LOW
- U1 pad 4: /SEG5_LOW -> /SEG3_LOW
- U1 pad 5: /SEG6_LOW -> /SEG4_LOW
- U1 pad 6: /SEG7_LOW -> /SEG5_LOW
- U1 pad 7: /SEG8_LOW -> GND
- U1 pad 8: GND -> /SRCLK
- U1 pad 9: unconnected-(U1-QH'-Pad9) -> +5V
- U2 pad 9: +3.3V -> +5V
- U3 pad 1: unconnected-(U3-QB-Pad1) -> /SEG7_LOW
- U3 pad 10: +5V -> unconnected-(U3-Q4-Pad10)
- U3 pad 11: /SRCLK -> unconnected-(U3-Q5-Pad11)
- U3 pad 12: /SRCLK -> unconnected-(U3-Q6-Pad12)
- U3 pad 13: GND -> unconnected-(U3-Q7-Pad13)
- U3 pad 14: /SEG7_LOW -> +5V
- U3 pad 2: unconnected-(U3-QC-Pad2) -> +5V
- U3 pad 3: unconnected-(U3-QD-Pad3) -> /SEG9_LOW
- U3 pad 8: GND -> /SRCLK
- U3 pad 9: unconnected-(U3-QH'-Pad9) -> +5V
Routing:
- net +3.3V: track 138.2 -> 0.00 mm, vias 1 -> 0
- net /SEG9_HIGH: track 179.5 -> 47.9 mm, vias 0 -> 1
- net /SEG8_HIGH: track 176.0 -> 47.9 mm, vias 0 -> 1
- net /SEG7_HIGH: track 170.3 -> 44.4 mm, vias 0 -> 1
- net /SEG1_LOW: track 111.7 -> 0.00 mm
- net /SER: track 112.3 -> 14.7 mm
- net /SEG6_HIGH: track 142.0 -> 58.5 mm, vias 1 -> 2
- net +5V: track 166.3 -> 84.1 mm
- net /SRCLK: track 116.3 -> 37.1 mm, vias 0 -> 2
- net /SEG4_LOW: track 90.0 -> 13.2 mm, vias 0 -> 2
- net /SEG5_HIGH: track 129.4 -> 59.9 mm, vias 1 -> 2
- net /F_HIGH: track 31.6 -> 99.4 mm
- net /SEG3_LOW: track 81.2 -> 15.9 mm, vias 1 -> 2
- net /SEG2_HIGH: track 0.00 -> 63.8 mm, vias 0 -> 2
- net /SEG2_LOW: track 77.8 -> 16.6 mm, vias 1 -> 2
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Other:
- board outline added: 100 x 70 mm
- board text added: "kill me pls <3"
- board text added: "uso.lovesyou.fr"
