File: pcb/e.kicad_sch (KiCad schematic)
At the start: 118 parts, among them J1 Grids and Anodes, J2 CH32V003 PROG, J3 AC 15V, J4 AC 27V, J5 AC Filament Middle, J6 Step-down IN, J7 Step-down OUT, J9 GPS Header, Q1 BC237, Q10 BC307, Q11 BC237, Q12 BC307, Q13 BC237, Q14 BC307, Q15 BC237, Q16 BC307, Q17 BC237, Q18 BC307, Q19 BC237, Q2 BC307, Q20 BC307, Q21 BC237, Q22 BC307, Q23 BC237, Q24 BC307, Q25 BC237, Q26 BC307, Q27 BC237, Q28 BC307, Q29 BC237, Q3 BC237, Q30 BC307, Q31 BC237, Q32 BC307, Q33 BC237, Q34 BC307, Q4 BC307, Q5 BC237, Q6 BC307, Q7 BC237, Q8 BC307, Q9 BC237, U1 74HC595, U2 CH32V003FxPx, U3 74HC595

Commit message: smd pcb
Parts:
- removed J6: Step-down IN, Connector_PinHeader_1.00mm:PinHeader_1x02_P1.00mm_Vertical, symbol Connector:Conn_01x02_Pin
- removed J7: Step-down OUT, Connector_PinHeader_1.00mm:PinHeader_1x02_P1.00mm_Vertical, symbol Connector:Conn_01x02_Pin
- added J10: GND, Connector_PinHeader_2.54mm:PinHeader_1x01_P2.54mm_Vertical, symbol Connector:Conn_01x01_Pin
- added J6: DC +15V, Connector_PinHeader_2.54mm:PinHeader_1x01_P2.54mm_Vertical, symbol Connector:Conn_01x01_Pin
- added J7: DC 15GND, Connector_PinHeader_2.54mm:PinHeader_1x01_P2.54mm_Vertical, symbol Connector:Conn_01x01_Pin
- added J8: DC +5V, Connector_PinHeader_2.54mm:PinHeader_1x01_P2.54mm_Vertical, symbol Connector:Conn_01x01_Pin
- Q1, Q11, Q13, Q15, Q17, Q19, Q21, Q23, Q25, Q27, Q29, Q3, Q31, Q33, Q5, Q7, Q9: value BC237 -> BC848; footprint Package_TO_SOT_THT:TO-92_Inline -> Package_TO_SOT_SMD:SOT-23; symbol Transistor_BJT:BC237 -> Transistor_BJT:BC848
- Q10, Q12, Q14, Q16, Q18, Q2, Q20, Q22, Q24, Q26, Q28, Q30, Q32, Q34, Q4, Q6, Q8: value BC307 -> BC856; footprint Package_TO_SOT_THT:TO-92_Inline -> Package_TO_SOT_SMD:SOT-23; symbol Transistor_BJT:BC307 -> Transistor_BJT:BC856
- R1, R10, R11, R12, R13, R14, R15, R16, R17, R18, R19, R2, R20, R21, R22, R23, R24, R25, R26, R27, R28, R29, R3, R30, R31, R32, R33, R34, R35, R36, R37, R38, R39, R4, R40, R41, R42, R43, R44, R45, R46, R47, R48, R49, R5, R50, R51, R52, R53, R54, R55, R56, R57, R58, R59, R6, R60, R61, R62, R63, R64, R65, R66, R67, R68, R7, R8, R9: footprint Resistor_THT:R_Axial_DIN0207_L6.3mm_D2.5mm_P10.16mm_Horizontal -> Resistor_SMD:R_0201_0603Metric
- U1, U3: value 74HC595 -> 74HC164; footprint Package_DIP:DIP-16_W7.62mm_Socket -> Package_SO:SSOP-14_5.3x6.2mm_P0.65mm; symbol 74xx:74HC595 -> 74xx:74HC164
Connections:
- net +5V: now also D1.1 (K), U1.14 (VCC), U1.2 (DSB), U1.9 (~{MR}), U2.9 (VDD), U3.14 (VCC), U3.2 (DSB), U3.9 (~{MR}); no longer U1.10 (~{SRCLR}), U3.10 (~{SRCLR})
- net A_HIGH: now also Q2.3 (C); no longer Q2.1 (C)
- net A_LOW: now also Q1.1 (B); no longer Q1.2 (B)
- net B_HIGH: now also Q4.3 (C); no longer Q4.1 (C)
- net B_LOW: now also Q3.1 (B); no longer Q3.2 (B)
- net C_HIGH: now also Q6.3 (C); no longer Q6.1 (C)
- net C_LOW: now also Q5.1 (B); no longer Q5.2 (B)
- net D_HIGH: now also Q8.3 (C); no longer Q8.1 (C)
- net D_LOW: now also Q7.1 (B); no longer Q7.2 (B)
- net E_HIGH: now also Q10.3 (C); no longer Q10.1 (C)
- net E_LOW: now also Q9.1 (B); no longer Q9.2 (B)
- net F_HIGH: now also Q12.3 (C); no longer Q12.1 (C)
- net F_LOW: now also Q11.1 (B); no longer Q11.2 (B)
- net GND: now also U1.7 (GND), J10.1 (Pin_1); no longer U1.13 (~{OE}), U1.8 (GND), U3.13 (~{OE}), U3.8 (GND)
- net G_HIGH: now also Q14.3 (C); no longer Q14.1 (C)
- net G_LOW: now also Q13.1 (B); no longer Q13.2 (B)
- net H_HIGH: now also Q16.3 (C); no longer Q16.1 (C)
- net H_LOW: now also Q15.1 (B); no longer Q15.2 (B)
- net SEG1_HIGH: now also Q18.3 (C); no longer Q18.1 (C), Q20.1 (C), R40.1
- net SEG1_LOW: now also Q17.1 (B); no longer Q17.2 (B), U1.15 (QA)
- net SEG2_HIGH: now also Q20.3 (C), R40.1
- net SEG2_LOW: now also Q19.1 (B), U1.3 (Q0); no longer Q19.2 (B), U1.1 (QB)
- net SEG3_HIGH: now also Q22.3 (C); no longer Q22.1 (C)
- net SEG3_LOW: now also Q21.1 (B), U1.4 (Q1); no longer Q21.2 (B), U1.2 (QC)
- net SEG4_HIGH: now also Q24.3 (C); no longer Q24.1 (C)
- net SEG4_LOW: now also Q23.1 (B), U1.5 (Q2); no longer Q23.2 (B), U1.3 (QD)
- net SEG5_HIGH: now also Q26.3 (C); no longer Q26.1 (C)
- net SEG5_LOW: now also Q25.1 (B), U1.6 (Q3); no longer Q25.2 (B), U1.4 (QE)
- net SEG6_HIGH: now also Q28.3 (C); no longer Q28.1 (C)
- net SEG6_LOW: now also Q27.1 (B), U1.10 (Q4); no longer Q27.2 (B), U1.5 (QF)
- net SEG7_HIGH: now also Q30.3 (C); no longer Q30.1 (C)
- net SEG7_LOW: now also Q29.1 (B), U1.11 (Q5), U3.1 (DSA); no longer Q29.2 (B), U1.6 (QG), U3.14 (SER)
- net SEG8_HIGH: now also Q32.3 (C); no longer Q32.1 (C)
- net SEG8_LOW: now also Q31.1 (B), U1.12 (Q6); no longer Q31.2 (B), U1.7 (QH)
- net SEG9_HIGH: now also Q34.3 (C); no longer Q34.1 (C)
- net SEG9_LOW: now also Q33.1 (B), U3.3 (Q0); no longer Q33.2 (B), U3.15 (QA)
- net SER: now also U1.1 (DSA); no longer U1.14 (SER)
- net SRCLK: now also U1.8 (CP), U3.8 (CP); no longer U1.11 (SRCLK), U1.12 (RCLK), U3.11 (SRCLK), U3.12 (RCLK)
- net at R63.2: now also Q32.2 (E); no longer Q32.3 (E)
- net at R54.1: now also Q27.2 (E); no longer Q27.3 (E)
- net at R22.1: now also Q11.2 (E); no longer Q11.3 (E)
- net at R19.2: now also Q10.2 (E); no longer Q10.3 (E)
- net at R58.1: now also Q29.2 (E); no longer Q29.3 (E)
- net at R10.1: now also Q5.2 (E); no longer Q5.3 (E)
- net at R66.1: now also Q33.2 (E); no longer Q33.3 (E)
- net at R31.2: now also Q16.2 (E); no longer Q16.3 (E)
- net at R42.1: now also Q21.2 (E); no longer Q21.3 (E)
- net at Q9.3 (C): now also Q10.1 (B), R17.2; no longer R18.1
- net at R59.2: now also Q30.2 (E); no longer Q30.3 (E)
- net at D1.2 (A): now also J8.1 (Pin_1)
- net at R7.2: now also Q4.2 (E); no longer Q4.3 (E)
- net at C2.1, D2.1 (+): now also J6.1 (Pin_1)
- net at C2.2, D2.4 (-): now also J7.1 (Pin_1)
- net at R50.1: now also Q25.2 (E); no longer Q25.3 (E)
- net at R43.2: now also Q22.2 (E); no longer Q22.3 (E)
- net at R15.2: now also Q8.2 (E); no longer Q8.3 (E)
- net at R26.1: now also Q13.2 (E); no longer Q13.3 (E)
- net at R27.2: now also Q14.2 (E); no longer Q14.3 (E)
- net at R23.2: now also Q12.2 (E); no longer Q12.3 (E)
- net at R39.2: now also Q20.2 (E); no longer Q20.3 (E)
- net at Q19.3 (C): now also Q20.1 (B), R37.2; no longer R38.1
- net at Q15.3 (C): now also Q16.1 (B), R29.2; no longer R30.1
- net at R35.2: now also Q18.2 (E); no longer Q18.3 (E)
- net at R11.2: now also Q6.2 (E); no longer Q6.3 (E)
- net at R2.2: now also Q2.2 (E); no longer Q2.3 (E)
- net at R51.2: now also Q26.2 (E); no longer Q26.3 (E)
- net at Q17.3 (C): now also Q18.1 (B), R33.2; no longer R34.1
- net at R67.2: now also Q34.2 (E); no longer Q34.3 (E)
- net at Q31.3 (C): now also Q32.1 (B), R61.2; no longer R62.1
- net at R55.2: now also Q28.2 (E); no longer Q28.3 (E)
- net at R3.1: now also Q1.2 (E); no longer Q1.3 (E)
- net at Q3.3 (C): now also Q4.1 (B), R5.2; no longer R6.1
- net at R47.2: now also Q24.2 (E); no longer Q24.3 (E)
- net at Q23.3 (C): now also Q24.1 (B), R45.2; no longer R46.1
- net at Q7.3 (C): now also Q8.1 (B), R13.2; no longer R14.1
- removed net +3.3V: D1.1 (K), U1.16 (VCC), U2.9 (VDD), U3.16 (VCC)
- new net: Q27.3 (C), Q28.1 (B), R53.2
- new net: Q5.3 (C), Q6.1 (B), R9.2
- new net: Q29.3 (C), Q30.1 (B), R57.2
- new net: Q33.3 (C), Q34.1 (B), R65.2
- new net: Q21.3 (C), Q22.1 (B), R41.2
- new net: Q9.2 (E), R18.1
- new net: Q11.3 (C), Q12.1 (B), R21.2
- new net: Q25.3 (C), Q26.1 (B), R49.2
- new net: Q19.2 (E), R38.1
- new net: Q15.2 (E), R30.1
- new net: Q13.3 (C), Q14.1 (B), R25.2
- new net: Q17.2 (E), R34.1
- new net: Q31.2 (E), R62.1
- new net: Q3.2 (E), R6.1
- new net: Q1.3 (C), Q2.1 (B), R1.2
- new net: Q23.2 (E), R46.1
- new net: Q7.2 (E), R14.1
